File: TMC4671-driver/V1.2.2_HALL/motor_board_tmc.sch (EAGLE design)
At the start: 164 parts, among them U1 TMC4671, U10 BSC030N08NS5ATMA1, U11 BSC030N08NS5ATMA1, U12 BSC030N08NS5ATMA1, U13 BSC030N08NS5ATMA1, U14 MCP14XX, U15 BSC030N08NS5ATMA1, U16 BSC030N08NS5ATMA1, U17 BSC030N08NS5ATMA1, U18 NC7NZ17K8X-3-BUFFER, U19 NC7NZ17K8X-3-BUFFER, U2 LM5109BSD, U20 LM74700-Q1, U22 BSC030N08NS5ATMA1, U23 MAX5033BASA+T, U24 AP3012KTR-G1, U3 LM5109BSD, U4 LM5109BSD, U5 LM5109BSD, U6 BSC030N08NS5ATMA1, U7 BSC030N08NS5ATMA1, U8 AD841X, U9 AD841X, X1 2516-, X2 GMSTBA4, X3 GMSTBA4, Y1 25MHz

Commit message: Added files for Hall sensor TMC
Parts:
- removed C40: 4.7µF, resistor:C-EUC0805
- removed C41, C42: 100nF, resistor:C-EUC0603
- removed C43: 1µF, resistor:C-EUC1206
- removed C44: 593D476X0016D2TE3, Powermisc:593D476X0016D2TE3
- removed C45: 4.7µF <REMOVE>, resistor:C-EUC0805
- removed R47: 294k, resistor:R-EU_R0805
- removed R48, R49: 71.5k, resistor:R-EU_R0805
- removed R50: 10k, resistor:R-EU_R0603
- removed R51: 33k, resistor:R-EU_R0603
- added D16: LV low drop, adafruit:DIODE_SOD-123FL
- added SJ5: (no value), jumper:SJ
- added SJ6: 3.3V, jumper:SJ
- C10, C9: value 100nF -> 680µF; device resistor:C-EUC0603 -> resistor:CPOL-EUE7.5-16
- C11, C12: value 680µF -> 1µF; device resistor:CPOL-EUE7.5-16 -> resistor:C-EUC1206
- C15, C16: value 1µF -> 100nF; device resistor:C-EUC1206 -> resistor:C-EUC0603
- C18: value 100nF -> 4.7µF; device resistor:C-EUC0603 -> resistor:C-EUC0805
- C20: value 4.7µF -> 100nF; device resistor:C-EUC0805 -> resistor:C-EUC0603
- C21, C22, C23, C24: device resistor:C-EUC0805 -> resistor:C-EUC0603
- C25: value 1n -> 4.7µF; device resistor:C-EUC0603 -> resistor:C-EUC0805
- C26: value 100nF -> 100n
- C27: value 100nF -> 1n
- C28: value 4.7µF -> 1n; device resistor:C-EUC0805 -> resistor:C-EUC0603
- C29: value (none) -> 1n; device resistor:CPOL-EUE5-8.5 -> resistor:C-EUC0603
- C32, C34: value 100p -> 4.7µF; device resistor:C-EUC0603 -> resistor:C-EUC0805
- C33, C35: value 1n -> 100nF
- C36: value 100p -> 100nF
- C37: value 1n -> 1µF; device resistor:C-EUC0603 -> resistor:C-EUC1206
- C38: value 4.7µF -> 593D476X0016D2TE3; device resistor:C-EUC0805 -> Powermisc:593D476X0016D2TE3
- C39: value 100nF -> 4.7µF
- D10: value BZX384-XXX -> LV low drop; device Powermisc:BZX384-XXX -> adafruit:DIODE_SOD-123FL
- D11: value HV >100V -> BZX384-XXX; device adafruit:DIODE_SOD-123FL -> Powermisc:BZX384-XXX
- D13: value 5.6V zener -> Zener 65V (MMSZ5265BT1G)
- D14: value LV low drop -> HV >100V
- D15: value Zener 65V (MMSZ5265BT1G) -> 5.6V zener
- JP1: device pinhead:PINHD-1X1 -> pinhead:PINHD-1X2
- R1, R19, R4: value 10k -> 2.2
- R12: value 2.2 -> 33k
- R13: value 71.5k -> 33k; device resistor:R-EU_R0805 -> resistor:R-EU_R0603
- R14: value 1.5k -> 33k
- R15, R18: value 294k -> 10k; device resistor:R-EU_R0805 -> resistor:R-EU_R0603
- R16: value 10k -> 1.5k
- R17, R28: value 33k -> 10k
- R21: value 1.5m -> 33k; device resistor:R-EU_R2512 -> resistor:R-EU_R0603
- R22: value 1.5m -> 1.5k; device resistor:R-EU_R2512 -> resistor:R-EU_R0603
- R23, R44, R45: value 1.5k -> 71.5k; device resistor:R-EU_R0603 -> resistor:R-EU_R0805
- R25: value 33k -> 294k; device resistor:R-EU_R0603 -> resistor:R-EU_R0805
- R27, R43: value 1.5k -> 294k; device resistor:R-EU_R0603 -> resistor:R-EU_R0805
- R29: value 22k thermistor -> 1.5k
- R30: value 1.5k -> 10k thermistor
- R32: value 10k -> 71.5k; device resistor:R-EU_R0603 -> resistor:R-EU_R0805
- R33: value 10k -> 47k
- R34: value 330 -> 4.7k
- R40: value 4.7k -> 1.5k
- R46: value 1.5k -> 10k
- SJ4: value 3.3V -> (none)
- U18: value NC7NZ17K8X-3-BUFFER -> MCP6004; device Powermisc:NC7NZ17K8X-3-BUFFER -> Powermisc:MCP6004
- U19: value NC7NZ17K8X-3-BUFFER -> 74LV17APWJ; device Powermisc:NC7NZ17K8X-3-BUFFER -> Powermisc:74LV17APWJ
- U6, U7: value BSC030N08NS5ATMA1 -> TMCS1100; device OHSC_Power:BSC030N08NS5ATMA1 -> Powermisc:TMCS1100
- U8, U9: value AD841X -> BSC030N08NS5ATMA1; device Powermisc:AD841X -> OHSC_Power:BSC030N08NS5ATMA1
Connections:
- removed net N$10: R24.2, U9.OUT
- removed net N$11: JP11.2, R35.1, R44.2
- removed net N$22: JP3.2, JP3.4, JP3.6, R32.1, R33.2
- removed net N$6: R23.2, U8.OUT
- removed net N$7: JP11.4, R38.1, R46.2
- removed net N$9: JP11.3, R36.1, R45.2
- removed net V_SENSE/2: C1.2, C2.2, R1.1, R2.2, U1A.ADC_I0_NEG, U1A.ADC_I1_NEG, U8.REF1, U8.REF2, U9.REF1, U9.REF2
- new net 2.5V_REF: C26.1, JP3.2, JP3.4, JP3.6, R30.2, SJ1.1, SJ2.1, U18.INB-, U18.OUTB
- new net 2.5V_REF_A: C27.1, SJ1.2, U1A.ADC_I0_NEG, U6.VREF
- new net 2.5V_REF_C: C28.1, SJ2.2, U1A.ADC_I1_NEG, U7.VREF
- new net 2.5V_REF_RAW: R17.1, R18.2, U18.INB+
- new net 5V_ADC: C2.2, R1.1, U1B.V5
- new net 5V_SENSE: C23.2, C24.1, C25.1, R17.2, R19.1, U18.VCC, U6.VS, U7.VS
- new net BRAKE_RES_COMP: D10.A, U18.OUTD
- new net BRAKE_RES_TH: R32.1, R33.2, U18.IND-
- new net TH_FET: R30.1, R31.2, U18.INA+
- new net V_INT_TMC_RAW: R23.1, R24.2, U18.INC+
- net +3V3: now also C15.1, C16.1, C34.1, R2.2, R32.2, SJ6.2; no longer C19.1, C20.1, C40.1, R3.2, R34.2, SJ4.2, U18.VCC
- net +5V: now also C32.1, D15.C, R19.2, R34.2; no longer C26.1, C27.1, C28.1, C29.+, C4.2, C44.1, D13.C, R32.2, R40.2, U1B.V5, U8.V+, U9.V+
- net AGPI_A: now also JP1.2; no longer JP1.1
- net AGPI_B: now also U18.INA-, U18.OUTA; no longer R29.1, R30.2
- net BRAKE_CTRL: now also D10.C, R15.2, R16.2; no longer R26.2, R27.2
- net BRAKE_CTRL_EXT: now also R16.1; no longer R27.1
- net BRAKE_GATE: now also R21.2; no longer R51.2
- net CS1: now also SJ3.1; no longer SJ1.1
- net CS2: now also SJ4.1; no longer SJ2.1
- net CS3: now also SJ5.1; no longer SJ3.1
- net CS_TMC: now also SJ4.2, SJ5.2; no longer SJ1.2, SJ2.2
- net ENABLE: now also R22.1; no longer R31.1
- net ENC_A: now also U19.3Y; no longer U18.3Y
- net ENC_A_5V: now also JP11.4, R37.1, U19.3A; no longer C36.2, R46.1, U18.3A
- net ENC_B: now also U19.2Y; no longer U18.2Y
- net ENC_B_5V: now also JP11.3, R35.1, U19.2A; no longer C34.2, R45.1, U18.2A
- net ENC_Z: now also U19.1Y; no longer U18.1Y
- net ENC_Z_5V: now also JP11.2, R34.1, U19.1A; no longer C32.2, R44.1, U18.1A
- net ENO: now also JP1.1
- net FLAG: now also R3.2; no longer R4.2
- net GND: now also C10.-, C11.2, C12.2, C23.1, C24.2, C29.1, C32.2, C34.2, C39.2, C9.-, D14.A, R12.1, R13.1, R15.1, R18.1, R21.1, R24.1, R3.1, R31.1, R44.2, R46.1, U6.GND, U7.GND, U9.S; no longer C10.1, C11.-, C12.-, C19.2, C20.2, C27.2, C28.2, C29.-, C32.1, C33.1, C34.1, C36.1, C40.2, C41.1, C43.1, C44.2, C45.2, C9.1, D12.A, R16.1, R17.1, R19.1, R2.1, R25.1, R30.1, R4.1, R48.2, R50.1, R51.1, U7.S, U8.GND, U9.GND
- net G_HS_A: now also R10.1, U8.G; no longer R11.1, U6.G
- net G_HS_B: now also R8.1; no longer R9.1
- net G_HS_C: now also R6.1; no longer R7.1
- net G_HS_D: now also D11.C, R4.1; no longer D10.C, R5.1
- net G_LS_A: now also R11.1, R12.2, U9.G; no longer R12.1, R17.2, U7.G
- net G_LS_B: now also R13.2, R9.1; no longer R10.1, R20.2
- net G_LS_C: now also R14.2, R7.1; no longer R25.2, R8.1
- net G_LS_D: now also R20.2, R5.1; no longer R28.2, R6.1
- net HALL_UX: now also U19.6Y; no longer U19.3Y
- net HALL_UX_5V: now also C29.2, R40.1, U19.6A; no longer C33.2, R41.1, U19.3A
- net HALL_V: now also U19.5Y; no longer U19.2Y
- net HALL_V_5V: now also C30.2, R41.1, U19.5A; no longer C35.2, R42.1, U19.2A
- net HALL_WY: now also U19.4Y; no longer U19.1Y
- net HALL_WY_5V: now also C31.2, R42.1, U19.4A; no longer C37.2, R43.1, U19.1A
- net MOT_A: now also C22.2, U6.IN+, U6.IN+_2, U8.S, U9.D; no longer C24.2, R22.2, U6.S, U7.D, U8.IN+
- net MOT_A_OUT: now also U6.IN-, U6.IN-_2; no longer R22.1, U8.IN-
- net MOT_B: now also C21.2; no longer C23.2
- net MOT_C: now also C20.2, U7.IN+, U7.IN+_2; no longer C22.2, R21.2, U9.IN+
- net MOT_C_OUT: now also U7.IN-, U7.IN-_2; no longer R21.1, U9.IN-
- net MOT_D: now also C19.2, D11.A; no longer C21.2, D10.A
- net N$1: now also R36.1, R40.2; no longer R37.1, R41.2
- net N$12: now also D16.A; no longer D14.A
- net N$13: now also R11.2; no longer R12.2
- net N$15: now also R39.1, R42.2; no longer R40.1, R43.2
- net N$16: now also C36.2, D14.C; no longer C42.2, D12.C
- net N$17: now also R22.2; no longer R31.2
- net N$18: now also C22.1; no longer C24.1
- net N$19: now also C36.1; no longer C42.1
- net N$20: now also SJ6.1; no longer SJ4.1
- net N$21: now also R43.1, R44.1; no longer R47.1, R48.1
- net N$24: now also C33.1; no longer C39.1
- net N$25: now also C35.2; no longer C41.2
- net N$27: now also R10.2; no longer R11.2
- net N$28: now also C21.1; no longer C23.1
- net N$29: now also R9.2; no longer R10.2
- net N$3: now also R38.1, R41.2; no longer R39.1, R42.2
- net N$30: now also R8.2; no longer R9.2
- net N$31: now also C19.1; no longer C21.1
- net N$32: now also R5.2; no longer R6.2
- net N$33: now also R4.2; no longer R5.2
- net N$34: now also C20.1; no longer C22.1
- net N$35: now also R7.2; no longer R8.2
- net N$36: now also R6.2; no longer R7.2
- net N$5: now also R45.1, R46.2; no longer R49.1, R50.2
- net N$8: now also R29.1; no longer R34.1
- net RESET: now also R2.1; no longer R3.1
- net RES_FET: now also D12.A, D13.C; no longer D11.A, D15.C
- net SENSE_A: now also C27.2, U6.VOUT; no longer C30.2, R23.1
- net SENSE_C: now also C28.2, U7.VOUT; no longer C31.2, R24.1
- net V+: now also C10.+, C11.1, C12.1, C37.2, C9.+, D12.C, R23.2, R25.2, R43.2, U8.D; no longer C11.+, C12.+, C15.1, C16.1, C43.2, D11.C, R13.2, R15.2, R47.2, U6.D
- net VCORE: now also C1.2, C4.2; no longer C5.2, C6.2
- net V_EXT: now also R27.1, R28.2; no longer R18.1, R19.2
- net V_GD: now also C39.1, C5.2, C6.2, D16.C, R45.2; no longer C10.2, C45.1, C9.2, D14.C, R49.2
- net V_INT: now also R25.1, R26.2; no longer R15.1, R16.2
- net V_INT_TMC: now also U18.INC-, U18.IND+, U18.OUTC; no longer C25.1, R13.1, R14.2
- net V_MOT_IN: now also C33.2, R27.2; no longer C39.2, R18.2
Other:
- note added: "1.3V"
- note added: "60V=>1.25V 65V=>1.336"
- note added: "Brake resistor forced activation point"
- note added: "Input 5V -> 3.3V buffer"
- note added: "Limit should be set to 1.7V max! Linear range up to 1.25V"
- note added: "MCP6004 or MCP6009"
- note added: "SHORT for TMCS1100, DISCONNECT for LEM GO SME"
- note added: "Supply filter analog"
- note added: "Thermistor 10k"
- note removed: "60V=>1.25V"
- note removed: "Optional filters"
- note removed: "Options: 20x gain + 3mOhm = 30A 60x + 1.5mOhm = 20A 60x + 1mOhm = 30A"
- note removed: "Thermistor 22k"
- note removed: "ad8417 (60x Gain) ad8418 (20x Gain)"
