File: OpenFFBoard-main/V1.2.4 F407/KiCad/OpenFFBoard-main.kicad_sch (KiCad schematic)
At the start: 64 parts, among them J1 USB4105-GF-A, SW1 TL3342F160QG{slash}TR, SW2 TL3342F160QG{slash}TR, U1 STM32F407VGT6, U2 TJA1051T{slash}3, U3 LM1117, U4 USBLC6-2SC6, X1 8MHz

Commit message: Consistent naming convention and font size on schematic
Parts:
- R1, R14, R5, R8: value 10k -> 10kR
- R10, R11, R12, R15, R16: value 5.1k -> 5.1kR
- R13: value 120 -> 120R
- R2, R3: value 22 -> 22R
- R4: value 1k -> 1kR
- R6, R7, R9: value 330 -> 330R
Other:
- moved on the sheet: JP11
